File: Build.kicad_pcb (KiCad board)
At the start: 2 copper layers, 285.8 x 95.2 mm, 149 parts, among them SW1 SW_Push, U1 ATmega32U4-AU, Y1 16MHz

Commit message: changed mounting side mounting holes
Parts:
- removed G*** (x2): LOGO, acheron_MountingHoles:halfSideHole
- added REF**: MountingHole_2.2mm_M2_Pad, MountingHole:MountingHole_2.2mm_M2_Pad, F.Cu at (299.4, 73.3)
- added REF**: MountingHole_2.2mm_M2_Pad, MountingHole:MountingHole_2.2mm_M2_Pad, F.Cu at (15.9, 73.3)
Changed lines of the file:
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@@
     (mod_text_size 1 1)
     (mod_text_width 0.15)
-    (pad_size 4.4 4.4)
-    (pad_drill 2.2)
+    (pad_size 10 4.5)
+    (pad_drill 8)
     (pad_to_mask_clearance 0.051)
     (solder_mask_min_width 0.25)
@@
   )
   (module MountingHole:MountingHole_2.2mm_M2_Pad (layer F.Cu)
+    (at 299.4025 73.279)
+    (descr "Mounting Hole 2.2mm, M2")
+    (tags "mounting hole 2.2mm m2")
+    (attr virtual)
+    (fp_text reference REF** (at 0 -3.2) (layer F.SilkS) hide
+      (effects (font (size 1 1) (thickness 0.15)))
+    )
+    (fp_text value MountingHole_2.2mm_M2_Pad (at 0 3.2) (layer F.Fab) hide
+      (effects (font (size 1 1) (thickness 0.15)))
+    )
+    (fp_circle (center 0 0) (end 2.45 0) (layer F.CrtYd) (width 0.05))
+    (fp_circle (center 0 0) (end 2.2 0) (layer Cmts.User) (width 0.15))
+    (fp_text user %R (at 0.3 0) (layer F.Fab)
+      (effects (font (size 1 1) (thickness 0.15)))
+    )
+    (pad 1 thru_hole oval (at 0 0) (size 10 4.5) (drill oval 8 2.5) (layers *.Cu *.Mask))
+  )
+  (module MountingHole:MountingHole_2.2mm_M2_Pad (layer F.Cu)
+    (at 15.9385 73.279)
+    (descr "Mounting Hole 2.2mm, M2")
+    (tags "mounting hole 2.2mm m2")
+    (attr virtual)
+    (fp_text reference REF** (at 0 -3.2) (layer F.SilkS) hide
+      (effects (font (size 1 1) (thickness 0.15)))
+    )
+    (fp_text value MountingHole_2.2mm_M2_Pad (at 0 3.2) (layer F.Fab) hide
+      (effects (font (size 1 1) (thickness 0.15)))
+    )
+    (fp_text user %R (at 0.3 0) (layer F.Fab)
+      (effects (font (size 1 1) (thickness 0.15)))
+    )
+    (fp_circle (center 0 0) (end 2.2 0) (layer Cmts.User) (width 0.15))
+    (fp_circle (center 0 0) (end 2.45 0) (layer F.CrtYd) (width 0.05))
+    (pad 1 thru_hole oval (at 0 0) (size 10 4.5) (drill oval 8 2.5) (layers *.Cu *.Mask))
+  )
+  (module MountingHole:MountingHole_2.2mm_M2_Pad (layer F.Cu)
     (at 271.907 44.577)
     (descr "Mounting Hole 2.2mm, M2")
@@
     (pad 1 thru_hole circle (at 0 0) (size 4.4 4.4) (drill 2.2) (layers *.Cu *.Mask))
   )
-  (module acheron_MountingHoles:halfSideHole (layer F.Cu)
-    (at 299.4025 73.279)
-    (fp_text reference G*** (at 3 -5) (layer Edge.Cuts) hide
-      (effects (font (size 1.524 1.524) (thickness 0.3)))
-    )
-    (fp_text value LOGO (at 3 5) (layer Edge.Cuts) hide
-      (effects (font (size 1.524 1.524) (thickness 0.3)))
-    )
-    (fp_line (start -6 0) (end 6 0) (layer Cmts.User) (width 0.1))
-    (fp_line (start 0 -4) (end 0 4) (layer Cmts.User) (width 0.1))
-    (pad "" thru_hole oval (at 0 0) (size 10 4.5) (drill oval 8 2.5) (layers *.Cu *.Mask))
-  )
-  (module acheron_MountingHoles:halfSideHole (layer F.Cu)
-    (at 15.9385 73.279)
-    (fp_text reference G*** (at 3 -5) (layer Edge.Cuts) hide
-      (effects (font (size 1.524 1.524) (thickness 0.3)))
-    )
-    (fp_text value LOGO (at 3 5) (layer Edge.Cuts) hide
-      (effects (font (size 1.524 1.524) (thickness 0.3)))
-    )
-    (fp_line (start -6 0) (end 6 0) (layer Cmts.User) (width 0.1))
-    (fp_line (start 0 -4) (end 0 4) (layer Cmts.User) (width 0.1))
-    (pad "" thru_hole oval (at 0 0) (size 10 4.5) (drill oval 8 2.5) (layers *.Cu *.Mask))
-  )
   (module MX_Only:MXOnly-2.25U-NoLED (layer F.Cu)

Commit message: Revert "changed mounting side mounting holes"
This reverts commit 6acce158d2db27eab7de2772cbacfb22acc69852.
Parts:
- removed the REF** at (299.4, 73.3)
- removed the REF** at (15.9, 73.3)
- added G***: LOGO, acheron_MountingHoles:halfSideHole, F.Cu at (299.4, 73.3)
- added G***: LOGO, acheron_MountingHoles:halfSideHole, F.Cu at (15.9, 73.3)
Changed lines of the file:
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@@
     (mod_text_size 1 1)
     (mod_text_width 0.15)
-    (pad_size 10 4.5)
-    (pad_drill 8)
+    (pad_size 4.4 4.4)
+    (pad_drill 2.2)
     (pad_to_mask_clearance 0.051)
     (solder_mask_min_width 0.25)
@@
   )
   (module MountingHole:MountingHole_2.2mm_M2_Pad (layer F.Cu)
-    (at 299.4025 73.279)
-    (descr "Mounting Hole 2.2mm, M2")
-    (tags "mounting hole 2.2mm m2")
-    (attr virtual)
-    (fp_text reference REF** (at 0 -3.2) (layer F.SilkS) hide
-      (effects (font (size 1 1) (thickness 0.15)))
-    )
-    (fp_text value MountingHole_2.2mm_M2_Pad (at 0 3.2) (layer F.Fab) hide
-      (effects (font (size 1 1) (thickness 0.15)))
-    )
-    (fp_circle (center 0 0) (end 2.45 0) (layer F.CrtYd) (width 0.05))
-    (fp_circle (center 0 0) (end 2.2 0) (layer Cmts.User) (width 0.15))
-    (fp_text user %R (at 0.3 0) (layer F.Fab)
-      (effects (font (size 1 1) (thickness 0.15)))
-    )
-    (pad 1 thru_hole oval (at 0 0) (size 10 4.5) (drill oval 8 2.5) (layers *.Cu *.Mask))
-  )
-  (module MountingHole:MountingHole_2.2mm_M2_Pad (layer F.Cu)
-    (at 15.9385 73.279)
-    (descr "Mounting Hole 2.2mm, M2")
-    (tags "mounting hole 2.2mm m2")
-    (attr virtual)
-    (fp_text reference REF** (at 0 -3.2) (layer F.SilkS) hide
-      (effects (font (size 1 1) (thickness 0.15)))
-    )
-    (fp_text value MountingHole_2.2mm_M2_Pad (at 0 3.2) (layer F.Fab) hide
-      (effects (font (size 1 1) (thickness 0.15)))
-    )
-    (fp_text user %R (at 0.3 0) (layer F.Fab)
-      (effects (font (size 1 1) (thickness 0.15)))
-    )
-    (fp_circle (center 0 0) (end 2.2 0) (layer Cmts.User) (width 0.15))
-    (fp_circle (center 0 0) (end 2.45 0) (layer F.CrtYd) (width 0.05))
-    (pad 1 thru_hole oval (at 0 0) (size 10 4.5) (drill oval 8 2.5) (layers *.Cu *.Mask))
-  )
-  (module MountingHole:MountingHole_2.2mm_M2_Pad (layer F.Cu)
     (at 271.907 44.577)
     (descr "Mounting Hole 2.2mm, M2")
@@
     (pad 1 thru_hole circle (at 0 0) (size 4.4 4.4) (drill 2.2) (layers *.Cu *.Mask))
   )
+  (module acheron_MountingHoles:halfSideHole (layer F.Cu)
+    (at 299.4025 73.279)
+    (fp_text reference G*** (at 3 -5) (layer Edge.Cuts) hide
+      (effects (font (size 1.524 1.524) (thickness 0.3)))
+    )
+    (fp_text value LOGO (at 3 5) (layer Edge.Cuts) hide
+      (effects (font (size 1.524 1.524) (thickness 0.3)))
+    )
+    (fp_line (start -6 0) (end 6 0) (layer Cmts.User) (width 0.1))
+    (fp_line (start 0 -4) (end 0 4) (layer Cmts.User) (width 0.1))
+    (pad "" thru_hole oval (at 0 0) (size 10 4.5) (drill oval 8 2.5) (layers *.Cu *.Mask))
+  )
+  (module acheron_MountingHoles:halfSideHole (layer F.Cu)
+    (at 15.9385 73.279)
+    (fp_text reference G*** (at 3 -5) (layer Edge.Cuts) hide
+      (effects (font (size 1.524 1.524) (thickness 0.3)))
+    )
+    (fp_text value LOGO (at 3 5) (layer Edge.Cuts) hide
+      (effects (font (size 1.524 1.524) (thickness 0.3)))
+    )
+    (fp_line (start -6 0) (end 6 0) (layer Cmts.User) (width 0.1))
+    (fp_line (start 0 -4) (end 0 4) (layer Cmts.User) (width 0.1))
+    (pad "" thru_hole oval (at 0 0) (size 10 4.5) (drill oval 8 2.5) (layers *.Cu *.Mask))
+  )
   (module MX_Only:MXOnly-2.25U-NoLED (layer F.Cu)

Commit message: changed side mounting holes
Parts:
- removed G*** (x2): LOGO, acheron_MountingHoles:halfSideHole
- added REF**: MountingHole_2.2mm_M2_Pad, MountingHole:MountingHole_2.2mm_M2_Pad, F.Cu at (299.3, 73.3)
- added REF**: MountingHole_2.2mm_M2_Pad, MountingHole:MountingHole_2.2mm_M2_Pad, F.Cu at (16.0, 73.3)
Changed lines of the file:
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@@
     (mod_text_size 1 1)
     (mod_text_width 0.15)
-    (pad_size 4.4 4.4)
-    (pad_drill 2.2)
+    (pad_size 10 4.5)
+    (pad_drill 8)
     (pad_to_mask_clearance 0.051)
     (solder_mask_min_width 0.25)
@@
   )
   (module MountingHole:MountingHole_2.2mm_M2_Pad (layer F.Cu)
+    (at 299.339 73.279)
+    (descr "Mounting Hole 2.2mm, M2")
+    (tags "mounting hole 2.2mm m2")
+    (attr virtual)
+    (fp_text reference REF** (at 0 -3.2) (layer F.SilkS) hide
+      (effects (font (size 1 1) (thickness 0.15)))
+    )
+    (fp_text value MountingHole_2.2mm_M2_Pad (at 0 3.2) (layer F.Fab) hide
+      (effects (font (size 1 1) (thickness 0.15)))
+    )
+    (fp_circle (center 0 0) (end 2.45 0) (layer F.CrtYd) (width 0.05))
+    (fp_circle (center 0 0) (end 2.2 0) (layer Cmts.User) (width 0.15))
+    (fp_text user %R (at 0.3 0) (layer F.Fab)
+      (effects (font (size 1 1) (thickness 0.15)))
+    )
+    (pad 1 thru_hole oval (at 0 0) (size 10 4.5) (drill oval 8 2.5) (layers *.Cu *.Mask))
+  )
+  (module MountingHole:MountingHole_2.2mm_M2_Pad (layer F.Cu)
+    (at 16.002 73.279)
+    (descr "Mounting Hole 2.2mm, M2")
+    (tags "mounting hole 2.2mm m2")
+    (attr virtual)
+    (fp_text reference REF** (at 0 -3.2) (layer F.SilkS) hide
+      (effects (font (size 1 1) (thickness 0.15)))
+    )
+    (fp_text value MountingHole_2.2mm_M2_Pad (at 0 3.2) (layer F.Fab) hide
+      (effects (font (size 1 1) (thickness 0.15)))
+    )
+    (fp_text user %R (at 0.3 0) (layer F.Fab)
+      (effects (font (size 1 1) (thickness 0.15)))
+    )
+    (fp_circle (center 0 0) (end 2.2 0) (layer Cmts.User) (width 0.15))
+    (fp_circle (center 0 0) (end 2.45 0) (layer F.CrtYd) (width 0.05))
+    (pad 1 thru_hole oval (at 0 0) (size 10 4.5) (drill oval 8 2.5) (layers *.Cu *.Mask))
+  )
+  (module MountingHole:MountingHole_2.2mm_M2_Pad (layer F.Cu)
     (at 271.907 44.577)
     (descr "Mounting Hole 2.2mm, M2")
@@
     (pad 1 thru_hole circle (at 0 0) (size 4.4 4.4) (drill 2.2) (layers *.Cu *.Mask))
   )
-  (module acheron_MountingHoles:halfSideHole (layer F.Cu)
-    (at 299.4025 73.279)
-    (fp_text reference G*** (at 3 -5) (layer Edge.Cuts) hide
-      (effects (font (size 1.524 1.524) (thickness 0.3)))
-    )
-    (fp_text value LOGO (at 3 5) (layer Edge.Cuts) hide
-      (effects (font (size 1.524 1.524) (thickness 0.3)))
-    )
-    (fp_line (start -6 0) (end 6 0) (layer Cmts.User) (width 0.1))
-    (fp_line (start 0 -4) (end 0 4) (layer Cmts.User) (width 0.1))
-    (pad "" thru_hole oval (at 0 0) (size 10 4.5) (drill oval 8 2.5) (layers *.Cu *.Mask))
-  )
-  (module acheron_MountingHoles:halfSideHole (layer F.Cu)
-    (at 15.9385 73.279)
-    (fp_text reference G*** (at 3 -5) (layer Edge.Cuts) hide
-      (effects (font (size 1.524 1.524) (thickness 0.3)))
-    )
-    (fp_text value LOGO (at 3 5) (layer Edge.Cuts) hide
-      (effects (font (size 1.524 1.524) (thickness 0.3)))
-    )
-    (fp_line (start -6 0) (end 6 0) (layer Cmts.User) (width 0.1))
-    (fp_line (start 0 -4) (end 0 4) (layer Cmts.User) (width 0.1))
-    (pad "" thru_hole oval (at 0 0) (size 10 4.5) (drill oval 8 2.5) (layers *.Cu *.Mask))
-  )
   (module MX_Only:MXOnly-2.25U-NoLED (layer F.Cu)
